Commit message: Update lidar.xacro

File: description/lidar.xacro (robot description, xacro)
@@ -7,5 +7,5 @@
         <origin xyz="0.122 0 0.09" rpy="0 0 0"/>
     </joint>
-    <link name="laser_frame">
+    <link name="laser">
         <visual>
             <geometry>
@@ -24,5 +24,5 @@
     </link>
     <!-- 2D Lidar Gazebo Sensor Plugin  -->
-    <gazebo reference="laser_frame">
+    <gazebo reference="laser">
         <material>Gazebo/Black</material>
         <sensor name="laser" type="ray">

Commit message: Update lidar.xacro

File: description/lidar.xacro (robot description, xacro)
@@ -4,5 +4,5 @@
     <joint name="laser_joint" type="fixed">
         <parent link="chassis"/>
-        <child link="laser_frame"/>
+        <child link="laser"/>
         <origin xyz="0.122 0 0.09" rpy="0 0 0"/>
     </joint>
